Commit message: clean of the repository

File: src/mybot/urdf/mybot.xacro (robot description, xacro)
@@ -3,7 +3,7 @@
   <xacro:property name="cameraSize" value="0.05"/>
   <xacro:property name="cameraMass" value="0.1"/>
-  <xacro:include filename="$(find mybot_description)/urdf/mybot.gazebo" />
-  <xacro:include filename="$(find mybot_description)/urdf/materials.xacro" />
-  <xacro:include filename="$(find mybot_description)/urdf/macros.xacro" />
+  <xacro:include filename="$(find mybot)/urdf/mybot.gazebo" />
+  <xacro:include filename="$(find mybot)/urdf/materials.xacro" />
+  <xacro:include filename="$(find mybot)/urdf/macros.xacro" />
   <link name='chassis'>
     <pose>0 0 0.1 0 0 0</pose>
@@ -181,5 +181,5 @@
       <origin xyz="0 0 0" rpy="0 0 0"/>
       <geometry>
-        <mesh filename="package://mybot_description/meshes/hokuyo.dae"/>
+        <mesh filename="package://mybot/meshes/hokuyo.dae"/>
       </geometry>
     </visual>

Commit message: clean only google-cartographer doesn't work

File: src/mybot/urdf/mybot.xacro (robot description, xacro)
@@ -5,188 +5,360 @@
   <xacro:include filename="$(find mybot)/urdf/mybot.gazebo" />
   <xacro:include filename="$(find mybot)/urdf/materials.xacro" />
-  <xacro:include filename="$(find mybot)/urdf/macros.xacro" />
-  <link name='chassis'>
-    <pose>0 0 0.1 0 0 0</pose>
-    <inertial>
-      <mass value="15.0"/>
-      <origin xyz="0.0 0 0.1" rpy=" 0 0 0"/>
-      <inertia
-          ixx="0.1" ixy="0" ixz="0"
-          iyy="0.1" iyz="0"
-          izz="0.1"
-      />
+<?xml version="1.0"?>
+<robot xmlns:sensor="http://playerstage.sourceforge.net/gazebo/xmlschema/#sensor"
+       xmlns:controller="http://playerstage.sourceforge.net/gazebo/xmlschema/#controller"
+       xmlns:interface="http://playerstage.sourceforge.net/gazebo/xmlschema/#interface"
+       xmlns:xacro="http://ros.org/wiki/xacro"
+name="pioneer3at">
+<!-- Chassis -->
+  <link name="base_link">
+    <!--  For pointers on inertial and gazebo-related parameters see
+           * http://wiki.ros.org/urdf/Tutorials/Adding%20Physical%20and%20Collision%20Properties%20to%20a%20URDF%20Model
+                       * http://answers.gazebosim.org/question/4372/the-inertia-matrix-explained/
+           * http://gazebosim.org/tutorials?tut=inertia&cat=build_robot, and
+                       * http://gazebosim.org/tutorials/?tut=ros_urdf
+                       * http://en.wikipedia.org/wiki/List_of_moment_of_inertia_tensors
+                -->
+    <inertial>
+      <mass value="21.5"/> <!-- P3AT 18.6kg plus three batteries @ 2.4kg each  minus four wheels @ 1.4 kg ea and top plate @ 0.1 kg-->
+      <origin xyz="-0.1 0 0.177"/>
+      <inertia ixx="0.3338" ixy="0.0"     ixz="0.0"
+                      iyy="0.4783"  iyz="0.0"
+                                    izz="0.3338"/>
     </inertial>
-    <collision name='collision'>
-      <geometry>
-        <box size=".4 .2 .1"/>
+    <visual>
+      <origin xyz="0 0 0.177" rpy="0 0 0"/>
+      <geometry name="pioneer_geom">
+        <mesh filename="package://amr_robots_description/meshes/p3at_meshes/chassis.stl"/>
       </geometry>
+      <material name="ChassisRed">
+        <color rgba="0.851 0.0 0.0 1.0"/>
+      </material>
+    </visual>
+    <collision>
+      <origin xyz="0 0 0.177" rpy="0 0 0"/>
+        <geometry>
+          <mesh filename="package://amr_robots_description/meshes/p3at_meshes/chassis.stl"/>
+        </geometry>
     </collision>
-    <visual name='chassis_visual'>
-      <origin xyz="0 0 0" rpy=" 0 0 0"/>
-      <geometry>
-        <box size=".4 .2 .1"/>
-      </geometry>
-    </visual>
-    <collision name='caster_collision'>
-      <origin xyz="-0.15 0 -0.05" rpy=" 0 0 0"/>
-      <geometry>
-        <sphere radius="0.05"/>
-      </geometry>
-      <surface>
-        <friction>
-          <ode>
-            <mu>0</mu>
-            <mu2>0</mu2>
-            <slip1>1.0</slip1>
-            <slip2>1.0</slip2>
-          </ode>
-        </friction>
-      </surface>
-    </collision>
-    <visual name='caster_visual'>
-      <origin xyz="-0.15 0 -0.05" rpy=" 0 0 0"/>
-      <geometry>
-        <sphere radius="0.05"/>
-      </geometry>
-    </visual>
-    <collision name='caster_front_collision'>
-      <origin xyz="0.15 0 -0.05" rpy=" 0 0 0"/>
-      <geometry>
-        <sphere radius="0.05"/>
-      </geometry>
-      <surface>
-        <friction>
-          <ode>
-            <mu>0</mu>
-            <mu2>0</mu2>
-            <slip1>1.0</slip1>
-            <slip2>1.0</slip2>
-          </ode>
-        </friction>
-      </surface>
-    </collision>
-    <visual name='caster_front_visual'>
-      <origin xyz="0.15 0 -0.05" rpy=" 0 0 0"/>
-      <geometry>
-        <sphere radius="0.05"/>
-      </geometry>
-    </visual>
-  </link>
-  <link name="left_wheel">
-    <!--origin xyz="0.1 0.13 0.1" rpy="0 1.5707 1.5707"/-->
-    <collision name="collision">
-      <origin xyz="0 0 0" rpy="0 1.5707 1.5707"/>
-      <geometry>
-        <cylinder radius="0.1" length="0.05"/>
-      </geometry>
-    </collision>
-    <visual name="left_wheel_visual">
-      <origin xyz="0 0 0" rpy="0 1.5707 1.5707"/>
-      <geometry>
-        <cylinder radius="0.1" length="0.05"/>
-      </geometry>
-    </visual>
-    <inertial>
-      <origin xyz="0 0 0" rpy="0 1.5707 1.5707"/>
-      <mass value="5"/>
-      <inertia
-        ixx=".1" ixy="0.0" ixz="0.0"
-        iyy=".1" iyz="0.0"
-        izz=".1"/>
+  </link>
+  <gazebo reference="base_link">
+    <material value="Gazebo/Red"/>
+  </gazebo>
+<!-- Top -->
+  <link name="top_plate">
+    <inertial>
+      <mass value="0.1"/>
+      <origin xyz="-0.025 0 -0.223"/>
+      <inertia ixx="1.0" ixy="0.0" ixz="0.0"
+         iyy="1.0" iyz="0.0"
+        izz="1.0"/>
     </inertial>
-  </link>
-  <link name="right_wheel">
-    <!--origin xyz="0.1 -0.13 0.1" rpy="0 1.5707 1.5707"/-->
-    <collision name="collision">
-      <origin xyz="0 0 0" rpy="0 1.5707 1.5707"/>
-      <geometry>
-        <cylinder radius="0.1" length="0.05"/>
-      </geometry>
-    </collision>
-    <visual name="right_wheel_visual">
-      <origin xyz="0 0 0" rpy="0 1.5707 1.5707"/>
-      <geometry>
-        <cylinder radius="0.1" length="0.05"/>
-      </geometry>
-    </visual>
-    <inertial>
-      <origin xyz="0 0 0" rpy="0 1.5707 1.5707"/>
-      <mass value="5"/>
-      <inertia
-        ixx=".1" ixy="0.0" ixz="0.0"
-        iyy=".1" iyz="0.0"
-        izz=".1"/>
-    </inertial>
-  </link>
-  <joint type="continuous" name="left_wheel_hinge">
-    <origin xyz="0 0.15 0" rpy="0 0 0"/>
-    <!--origin xyz="0.1 0.13 0" rpy="0 1.5707 1.5707"/-->
-    <child link="left_wheel"/>
-    <parent link="chassis"/>
-    <axis xyz="0 1 0" rpy="0 0 0"/>
-    <limit effort="10000" velocity="1000"/>
-    <joint_properties damping="1.0" friction="1.0"/>
-  </joint>
-  <joint type="continuous" name="right_wheel_hinge">
-    <origin xyz="0 -0.15 0" rpy="0 0 0"/>
-    <!--origin xyz="0.1 -0.13 0" rpy="0 1.5707 1.5707"/-->
-    <child link="right_wheel"/>
-    <parent link="chassis"/>
-    <axis xyz="0 1 0" rpy="0 0 0"/>
-    <limit effort="10000" velocity="1000"/>
-    <joint_properties damping="1.0" friction="1.0"/>
-  </joint>
-  <link name="camera">
-    <collision>
-      <origin xyz="0 0 0" rpy="0 0 0"/>
-      <geometry>
-        <box size="${cameraSize} ${cameraSize} ${cameraSize}"/>
-      </geometry>
-    </collision>
     <visual>
       <origin xyz="0 0 0" rpy="0 0 0"/>
-      <geometry>
-        <box size="${cameraSize} ${cameraSize} ${cameraSize}"/>
+      <geometry name="pioneer_geom">
+        <mesh filename="package://amr_robots_description/meshes/p3at_meshes/top.stl"/>
       </geometry>
-      <material name="green"/>
+      <material name="TopBlack">
+          <color rgba="0.038 0.038 0.038 1.0"/>
+      </material>
     </visual>
-    <inertial>
-      <mass value="${cameraMass}" />
-      <origin xyz="0 0 0" rpy="0 0 0"/>
-      <box_inertia m="${cameraMass}" x="${cameraSize}" y="${cameraSize}" z="${cameraSize}" />
-      <inertia ixx="1e-6" ixy="0" ixz="0" iyy="1e-6" iyz="0" izz="1e-6" />
+  </link>
+  <gazebo reference="top_plate">
+    <material>Gazebo/Black</material>
+  </gazebo>
+  <joint name="base_top_joint" type="fixed">
+    <origin xyz="0.003 0 0.274" rpy="0 0 0"/>
+    <parent link="base_link"/>
+    <child link="top_plate"/>
+  </joint>
+<!-- Front + Back Sonar -->
+  <link name="front_sonar">
+    <inertial>
+      <mass value="0.1"/>
+      <origin xyz="0 0 0"/>
+      <inertia ixx="1.0" ixy="0.0" ixz="0.0"
+         iyy="1.0" iyz="0.0" izz="1.0"/>
     </inertial>
-  </link>
-  <joint name="camera_joint" type="fixed">
-    <axis xyz="0 1 0" />
-    <origin xyz=".2 0 0" rpy="0 0 0"/>
-    <parent link="chassis"/>
-    <child link="camera"/>
-  </joint>
-  <joint name="hokuyo_joint" type="fixed">
-    <axis xyz="0 1 0" />
-    <origin xyz=".15 0 .1" rpy="0 0 0"/>
-    <parent link="chassis"/>
-    <child link="hokuyo"/>
-  </joint>
-  <!-- Hokuyo Laser -->
-  <link name="hokuyo">
-    <collision>
-      <origin xyz="0 0 0" rpy="0 0 0"/>
-      <geometry>
-    <box size="0.1 0.1 0.1"/>
-      </geometry>
-    </collision>
     <visual>
       <origin xyz="0 0 0" rpy="0 0 0"/>
-      <geometry>
-        <mesh filename="package://mybot/meshes/hokuyo.dae"/>
+      <geometry name="pioneer_geom">
+        <mesh filename="package://amr_robots_description/meshes/p3at_meshes/front_sonar.stl"/>
       </geometry>
+      <material name="SonarYellow">
+        <color rgba="0.715 0.583 0.210 1.0"/>
+      </material>
     </visual>
-    <inertial>
-      <mass value="1e-5" />
+  </link>
+  <gazebo reference="front_sonar">
+    <material value="Gazebo/Yellow"/>
+  </gazebo>
+  <joint name="base_front_joint" type="fixed">
+    <origin xyz="0.193 0 0.25" rpy="0 0 0"/>
+    <parent link="base_link"/>
+    <child link="front_sonar"/>
+  </joint>
+  <link name="back_sonar">
+    <inertial>
+      <mass value="0.1"/>
+      <origin xyz="0 0 0"/>
+      <inertia ixx="1.0" ixy="0.0" ixz="0.0"
+         iyy="1.0" iyz="0.0" izz="1.0"/>
+    </inertial>
+    <visual>
       <origin xyz="0 0 0" rpy="0 0 0"/>
-      <inertia ixx="1e-6" ixy="0" ixz="0" iyy="1e-6" iyz="0" izz="1e-6" />
-    </inertial>
-  </link>
+      <geometry name="pioneer_geom">
+        <mesh filename="package://amr_robots_description/meshes/p3at_meshes/back_sonar.stl"/>
+      </geometry>
+      <material name="SonarYellow">
+        <color rgba="0.715 0.583 0.210 1.0"/>
+      </material>
+    </visual>
+  </link>
+  <gazebo reference="back_sonar">
+    <material value="Gazebo/Yellow"/>
+  </gazebo>
+  <joint name="base_back_joint" type="fixed">
+    <origin xyz="-0.187 0 0.247" rpy="0 0 0"/>
+    <parent link="base_link"/>
+    <child link="back_sonar"/>
+  </joint>
+<xacro:macro name="p3at_drive_side" params="side reflect">
+  <!-- Front Axles + Wheels + Hubcaps -->
+  <link name="p3at_front_${side}_axle">
+    <inertial>
+      <mass value="0.1"/>
+      <origin xyz="0 0 0"/>
+      <inertia ixx="1.0" ixy="0.0" ixz="0.0"
+         iyy="1.0" iyz="0.0" izz="1.0"/>
+      </inertial>
+  <visual>
+    <origin xyz="0 0 0" rpy="0 0 0"/>
+    <geometry name="pioneer_geom">
+      <mesh filename="package://amr_robots_description/meshes/p3at_meshes/axle.stl"/>
+    </geometry>
+    <material name="AxleGrey">
+      <color rgba="0.5 0.5 0.5 1"/>
+    </material>
+  </visual>
+  </link>
+  <gazebo reference="p3at_front_${side}_axle">
+    <material value="Gazebo/Grey"/>
+  </gazebo>
+  <joint name="base_front_${side}_axle_joint" type="fixed">
+    <origin xyz="0.135 ${reflect*0.156} 0.111" rpy="0 0 0"/>
+    <parent link="base_link"/>
+    <child link="p3at_front_${side}_axle"/>
+  </joint>
+  <link name="p3at_front_${side}_hub">
+    <inertial>
+      <mass value="0.1"/>
+      <origin xyz="0 0 0"/>
+      <inertia ixx="1.0" ixy="0.0" ixz="0.0"
+         iyy="1.0" iyz="0.0" izz="1.0"/>
+      </inertial>
+  <visual>
+    <origin xyz="0 0 0" rpy="0 0 0"/>
+    <geometry name="pioneer_geom">
+      <mesh filename="package://amr_robots_description/meshes/p3at_meshes/${side}_hubcap.stl"/>
+    </geometry>
+    <material name="HubcapYellow">
+      <color rgba="1.0 0.811 0.151 1.0"/>
+    </material>
+  </visual>
+  </link>
+  <gazebo reference="p3at_front_${side}_hub">
+    <material value="Gazebo/Yellow"/>
+  </gazebo>
+  <joint name="base_front_${side}_hub_joint" type="fixed">
+    <origin xyz="0 ${reflect*0.041} 0" rpy="0 0 0"/>
+    <parent link="p3at_front_${side}_axle"/>
+    <child link="p3at_front_${side}_hub"/>
+  </joint>
+  <link name="p3at_front_${side}_wheel">
+    <inertial>
+      <mass value="1.2"/> <!-- 1.4 kg - axle 0.1 kg - hub 0.1 kg -->
+      <origin xyz="0 0 0"/>
+      <inertia ixx="0.012411765597" ixy="0" ixz="0"
+         iyy="0.015218160428" iyz="0" izz="0.011763977943"/>
+      </inertial>
+  <visual>
+    <origin xyz="0 0 0" rpy="0 0 0"/>
+    <geometry name="pioneer_geom">
+      <mesh filename="package://amr_robots_description/meshes/p3at_meshes/wheel.stl"/>
+    </geometry>
+    <material name="WheelBlack">
+      <color rgba="0.117 0.117 0.117 1"/>
+    </material>
+  </visual>
+  <collision>
+    <origin xyz="0 0 0" rpy="${-3.1415927/2} 0 0"/>
+    <geometry>
+      <!--mesh filename="package://amr_robots_description/meshes/p3at_meshes/wheel.stl"/-->
+      <cylinder radius="0.111" length="0.075"/>
+    </geometry>
+  </collision>
+  </link>
+  <gazebo reference="p3at_front_${side}_wheel">
+    <material value="Gazebo/Black"/>
+  </gazebo>
+  <joint name="p3at_front_${side}_wheel_joint" type="continuous">
+    <axis xyz="0 1 0"/>
+    <anchor xyz="0 0 0"/>
+    <limit effort="100" velocity="100" />
+    <joint_properties damping="0.7"/>
+    <origin xyz="0 0 0" rpy="0 0 0"/>
+    <parent link="p3at_front_${side}_hub"/>
+    <child link="p3at_front_${side}_wheel"/>
+  </joint>
+<!-- Back Axles + Wheels + Hubcaps -->
+  <link name="p3at_back_${side}_axle">
+    <inertial>
+      <mass value="0.1"/>
+      <origin xyz="0 0 0"/>
+      <inertia ixx="1.0" ixy="0.0" ixz="0.0"
+         iyy="1.0" iyz="0.0" izz="1.0"/>
+      </inertial>
+  <visual>
+    <origin xyz="0 0 0" rpy="0 0 0"/>
+    <geometry name="pioneer_geom">
+      <mesh filename="package://amr_robots_description/meshes/p3at_meshes/axle.stl"/>
+    </geometry>
+    <material name="AxleGrey">
+      <color rgba="0.5 0.5 0.5 1"/>
+    </material>
+  </visual>
+  <collision>
+    <origin xyz="0 0 0" rpy="0 0 0"/>
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