Commit message: hector localization working

File: src/mybot/urdf/mybot.xacro (robot description, xacro)
@@ -1,34 +1,22 @@
-<?xml version='1.0'?>
-<robot name="myrobot" xmlns:xacro="http://www.ros.org/wiki/xacro">
-  <xacro:property name="cameraSize" value="0.05"/>
-  <xacro:property name="cameraMass" value="0.1"/>
-  <xacro:include filename="$(find mybot)/urdf/mybot.gazebo" />
-  <xacro:include filename="$(find mybot)/urdf/materials.xacro" />
-<?xml version="1.0"?>
 <robot xmlns:sensor="http://playerstage.sourceforge.net/gazebo/xmlschema/#sensor"
        xmlns:controller="http://playerstage.sourceforge.net/gazebo/xmlschema/#controller"
        xmlns:interface="http://playerstage.sourceforge.net/gazebo/xmlschema/#interface"
        xmlns:xacro="http://ros.org/wiki/xacro"
-name="pioneer3at">
+name="pioneer3at"
+>
+<xacro:include filename="$(find mybot)/urdf/mybot.gazebo" />
 <!-- Chassis -->
   <link name="base_link">
-    <!--  For pointers on inertial and gazebo-related parameters see
-           * http://wiki.ros.org/urdf/Tutorials/Adding%20Physical%20and%20Collision%20Properties%20to%20a%20URDF%20Model
-                       * http://answers.gazebosim.org/question/4372/the-inertia-matrix-explained/
-           * http://gazebosim.org/tutorials?tut=inertia&cat=build_robot, and
-                       * http://gazebosim.org/tutorials/?tut=ros_urdf
-                       * http://en.wikipedia.org/wiki/List_of_moment_of_inertia_tensors
-                -->
-    <inertial>
-      <mass value="21.5"/> <!-- P3AT 18.6kg plus three batteries @ 2.4kg each  minus four wheels @ 1.4 kg ea and top plate @ 0.1 kg-->
-      <origin xyz="-0.1 0 0.177"/>
-      <inertia ixx="0.3338" ixy="0.0"     ixz="0.0"
-                      iyy="0.4783"  iyz="0.0"
-                                    izz="0.3338"/>
+    <inertial>
+      <mass value="10.0"/>
+      <origin xyz="0 0 0.177"/>
+      <inertia ixx="0.3338" ixy="0.0" ixz="0.0"
+         iyy="0.4783" iyz="0.0"
+         izz="0.3338"/>
     </inertial>
-    <visual>
+    <visual name="base_visual">
       <origin xyz="0 0 0.177" rpy="0 0 0"/>
       <geometry name="pioneer_geom">
-        <mesh filename="package://amr_robots_description/meshes/p3at_meshes/chassis.stl"/>
+        <mesh filename="package://mybot/meshes/p3at_meshes/chassis.stl"/>
       </geometry>
       <material name="ChassisRed">
@@ -39,5 +27,5 @@
       <origin xyz="0 0 0.177" rpy="0 0 0"/>
         <geometry>
-          <mesh filename="package://amr_robots_description/meshes/p3at_meshes/chassis.stl"/>
+          <mesh filename="package://mybot/meshes/p3at_meshes/chassis.stl"/>
         </geometry>
     </collision>
@@ -46,4 +34,19 @@
     <material value="Gazebo/Red"/>
   </gazebo>
+<!--link name="odom">
+</link>
+<joint name="odom_base" type="floating">
+    <origin xyz="0 0 0" rpy="0 0 0"/>
+    <parent link="odom"/>
+    <child link="base_link"/>
+  </joint-->
+<!--<link name="map">
+</link-->
+<!--<joint name="map_odom" type="fixed">
+    <origin xyz="0 0 0" rpy="0 0 0"/>
+    <parent link="map"/>
+    <child link="odom"/>
+  </joint>
+  -->
 <!-- Top -->
   <link name="top_plate">
@@ -55,8 +58,8 @@
         izz="1.0"/>
     </inertial>
-    <visual>
+    <visual name="base_visual">
       <origin xyz="0 0 0" rpy="0 0 0"/>
       <geometry name="pioneer_geom">
-        <mesh filename="package://amr_robots_description/meshes/p3at_meshes/top.stl"/>
+        <mesh filename="package://mybot/meshes/p3at_meshes/top.stl"/>
       </geometry>
       <material name="TopBlack">
@@ -64,7 +67,13 @@
       </material>
     </visual>
+    <collision>
+      <origin xyz="0 0 0" rpy="0 0 0"/>
+      <geometry>
+        <box size="0 0 0"/>
+      </geometry>
+    </collision>
   </link>
   <gazebo reference="top_plate">
-    <material>Gazebo/Black</material>
+    <material value="Gazebo/Black"/>
   </gazebo>
   <joint name="base_top_joint" type="fixed">
@@ -81,8 +90,8 @@
          iyy="1.0" iyz="0.0" izz="1.0"/>
     </inertial>
-    <visual>
+    <visual name="base_visual">
       <origin xyz="0 0 0" rpy="0 0 0"/>
       <geometry name="pioneer_geom">
-        <mesh filename="package://amr_robots_description/meshes/p3at_meshes/front_sonar.stl"/>
+        <mesh filename="package://mybot/meshes/p3at_meshes/front_sonar.stl"/>
       </geometry>
       <material name="SonarYellow">
@@ -90,4 +99,10 @@
       </material>
     </visual>
+    <collision>
+      <origin xyz="0 0 0" rpy="0 0 0"/>
+      <geometry>
+        <box size="0 0 0"/>
+      </geometry>
+    </collision>
   </link>
   <gazebo reference="front_sonar">
@@ -106,8 +121,8 @@
          iyy="1.0" iyz="0.0" izz="1.0"/>
     </inertial>
-    <visual>
+    <visual name="base_visual">
       <origin xyz="0 0 0" rpy="0 0 0"/>
       <geometry name="pioneer_geom">
-        <mesh filename="package://amr_robots_description/meshes/p3at_meshes/back_sonar.stl"/>
+        <mesh filename="package://mybot/meshes/p3at_meshes/back_sonar.stl"/>
       </geometry>
       <material name="SonarYellow">
@@ -115,4 +130,10 @@
       </material>
     </visual>
+    <collision>
+      <origin xyz="0 0 0" rpy="0 0 0"/>
+      <geometry>
+        <box size="0 0 0"/>
+      </geometry>
+    </collision>
   </link>
   <gazebo reference="back_sonar">
@@ -124,17 +145,17 @@
     <child link="back_sonar"/>
   </joint>
-<xacro:macro name="p3at_drive_side" params="side reflect">
-  <!-- Front Axles + Wheels + Hubcaps -->
-  <link name="p3at_front_${side}_axle">
-    <inertial>
-      <mass value="0.1"/>
-      <origin xyz="0 0 0"/>
-      <inertia ixx="1.0" ixy="0.0" ixz="0.0"
-         iyy="1.0" iyz="0.0" izz="1.0"/>
-      </inertial>
-  <visual>
-    <origin xyz="0 0 0" rpy="0 0 0"/>
-    <geometry name="pioneer_geom">
-      <mesh filename="package://amr_robots_description/meshes/p3at_meshes/axle.stl"/>
+<!-- Front Axles + Wheels + Hubcaps -->
+<xacro:macro name="p3at_front" params="suffix reflect">
+  <link name="p3at_front_${suffix}_axle">
+    <inertial>
+      <mass value="0.1"/>
+      <origin xyz="0 0 0"/>
+      <inertia ixx="1.0" ixy="0.0" ixz="0.0"
+         iyy="1.0" iyz="0.0" izz="1.0"/>
+      </inertial>
+  <visual name="base_visual">
+    <origin xyz="0 0 0" rpy="0 0 0"/>
+    <geometry name="pioneer_geom">
+      <mesh filename="package://mybot/meshes/p3at_meshes/axle.stl"/>
     </geometry>
     <material name="AxleGrey">
@@ -142,24 +163,30 @@
     </material>
   </visual>
-  </link>
-  <gazebo reference="p3at_front_${side}_axle">
+  <collision>
+    <origin xyz="0 0 0" rpy="0 0 0"/>
+    <geometry>
+      <box size="0 0 0"/>
+    </geometry>
+  </collision>
+  </link>
+  <gazebo reference="p3at_front_${suffix}_axle">
     <material value="Gazebo/Grey"/>
   </gazebo>
-  <joint name="base_front_${side}_axle_joint" type="fixed">
+  <joint name="base_front_${suffix}_axle_joint" type="fixed">
     <origin xyz="0.135 ${reflect*0.156} 0.111" rpy="0 0 0"/>
     <parent link="base_link"/>
-    <child link="p3at_front_${side}_axle"/>
-  </joint>
-  <link name="p3at_front_${side}_hub">
-    <inertial>
-      <mass value="0.1"/>
-      <origin xyz="0 0 0"/>
-      <inertia ixx="1.0" ixy="0.0" ixz="0.0"
-         iyy="1.0" iyz="0.0" izz="1.0"/>
-      </inertial>
-  <visual>
-    <origin xyz="0 0 0" rpy="0 0 0"/>
-    <geometry name="pioneer_geom">
-      <mesh filename="package://amr_robots_description/meshes/p3at_meshes/${side}_hubcap.stl"/>
+    <child link="p3at_front_${suffix}_axle"/>
+  </joint>
+  <link name="p3at_front_${suffix}_hub">
+    <inertial>
+      <mass value="0.1"/>
+      <origin xyz="0 0 0"/>
+      <inertia ixx="1.0" ixy="0.0" ixz="0.0"
+         iyy="1.0" iyz="0.0" izz="1.0"/>
+      </inertial>
+  <visual name="base_visual">
+    <origin xyz="0 0 0" rpy="0 0 0"/>
+    <geometry name="pioneer_geom">
+      <mesh filename="package://mybot/meshes/p3at_meshes/${suffix}_hubcap.stl"/>
     </geometry>
     <material name="HubcapYellow">
@@ -167,24 +194,30 @@
     </material>
   </visual>
-  </link>
-  <gazebo reference="p3at_front_${side}_hub">
+  <collision>
+    <origin xyz="0 0 0" rpy="0 0 0"/>
+    <geometry>
+      <box size="0 0 0"/>
+    </geometry>
+  </collision>
+  </link>
+  <gazebo reference="p3at_front_${suffix}_hub">
     <material value="Gazebo/Yellow"/>
   </gazebo>
-  <joint name="base_front_${side}_hub_joint" type="fixed">
+  <joint name="base_front_${suffix}_hub_joint" type="fixed">
     <origin xyz="0 ${reflect*0.041} 0" rpy="0 0 0"/>
-    <parent link="p3at_front_${side}_axle"/>
-    <child link="p3at_front_${side}_hub"/>
-  </joint>
-  <link name="p3at_front_${side}_wheel">
-    <inertial>
-      <mass value="1.2"/> <!-- 1.4 kg - axle 0.1 kg - hub 0.1 kg -->
+    <parent link="p3at_front_${suffix}_axle"/>
+    <child link="p3at_front_${suffix}_hub"/>
+  </joint>
+  <link name="p3at_front_${suffix}_wheel">
+    <inertial>
+      <mass value="0.5"/>
       <origin xyz="0 0 0"/>
       <inertia ixx="0.012411765597" ixy="0" ixz="0"
          iyy="0.015218160428" iyz="0" izz="0.011763977943"/>
       </inertial>
-  <visual>
-    <origin xyz="0 0 0" rpy="0 0 0"/>
-    <geometry name="pioneer_geom">
-      <mesh filename="package://amr_robots_description/meshes/p3at_meshes/wheel.stl"/>
+  <visual name="base_visual">
+    <origin xyz="0 0 0" rpy="0 0 0"/>
+    <geometry name="pioneer_geom">
+      <mesh filename="package://mybot/meshes/p3at_meshes/wheel.stl"/>
     </geometry>
     <material name="WheelBlack">
@@ -195,33 +228,33 @@
     <origin xyz="0 0 0" rpy="${-3.1415927/2} 0 0"/>
     <geometry>
-      <!--mesh filename="package://amr_robots_description/meshes/p3at_meshes/wheel.stl"/-->
+      <!--mesh filename="package://mybot/meshes/p3at_meshes/wheel.stl"/-->
       <cylinder radius="0.111" length="0.075"/>
     </geometry>
   </collision>
   </link>
-  <gazebo reference="p3at_front_${side}_wheel">
+  <gazebo reference="p3at_front_${suffix}_wheel">
     <material value="Gazebo/Black"/>
   </gazebo>
-  <joint name="p3at_front_${side}_wheel_joint" type="continuous">
-    <axis xyz="0 1 0"/>
-    <anchor xyz="0 0 0"/>
-    <limit effort="100" velocity="100" />
-    <joint_properties damping="0.7"/>
-    <origin xyz="0 0 0" rpy="0 0 0"/>
-    <parent link="p3at_front_${side}_hub"/>
-    <child link="p3at_front_${side}_wheel"/>
+  <joint name="p3at_front_${suffix}_wheel_joint" type="continuous">
+  <axis xyz="0 1 0"/>
+        <anchor xyz="0 0 0"/>
+  <origin xyz="0 0 0" rpy="0 0 0"/>
+  <parent link="p3at_front_${suffix}_hub"/>
+  <child link="p3at_front_${suffix}_wheel"/>
+        <limit effort="100" velocity="100" />
+        <joint_properties damping="0.7"/>
   </joint>
 <!-- Back Axles + Wheels + Hubcaps -->
-  <link name="p3at_back_${side}_axle">
-    <inertial>
-      <mass value="0.1"/>
-      <origin xyz="0 0 0"/>
-      <inertia ixx="1.0" ixy="0.0" ixz="0.0"
-         iyy="1.0" iyz="0.0" izz="1.0"/>
-      </inertial>
-  <visual>
-    <origin xyz="0 0 0" rpy="0 0 0"/>
-    <geometry name="pioneer_geom">
-      <mesh filename="package://amr_robots_description/meshes/p3at_meshes/axle.stl"/>
+  <link name="p3at_back_${suffix}_axle">
+    <inertial>
+      <mass value="0.1"/>
+      <origin xyz="0 0 0"/>
+      <inertia ixx="1.0" ixy="0.0" ixz="0.0"
+         iyy="1.0" iyz="0.0" izz="1.0"/>
+      </inertial>
+  <visual name="base_visual">
+    <origin xyz="0 0 0" rpy="0 0 0"/>
+    <geometry name="pioneer_geom">
+      <mesh filename="package://mybot/meshes/p3at_meshes/axle.stl"/>
     </geometry>
     <material name="AxleGrey">
@@ -232,27 +265,27 @@
     <origin xyz="0 0 0" rpy="0 0 0"/>
     <geometry>
-      <mesh filename="package://amr_robots_description/meshes/p3at_meshes/axle.stl"/>
-    </geometry>
-  </collision>
-  </link>
-  <gazebo reference="p3at_back_${side}_axle">
+      <mesh filename="package://mybot/meshes/p3at_meshes/axle.stl"/>
+    </geometry>
+  </collision>
+  </link>
+  <gazebo reference="p3at_back_${suffix}_axle">
     <material value="Gazebo/Grey"/>
   </gazebo>
-  <joint name="p3at_back_${side}_axle_joint" type="fixed">
+  <joint name="p3at_back_${suffix}_axle_joint" type="fixed">
     <origin xyz="-0.134 ${reflect*0.156} 0.111" rpy="0 0 0"/>
     <parent link="base_link"/>
-    <child link="p3at_back_${side}_axle"/>
-  </joint>
-  <link name="p3at_back_${side}_hub">
-    <inertial>
-      <mass value="0.1"/>
-      <origin xyz="0 0 0"/>
-      <inertia ixx="1.0" ixy="0.0" ixz="0.0"
-         iyy="1.0" iyz="0.0" izz="1.0"/>
-      </inertial>
-  <visual>
-    <origin xyz="0 0 0" rpy="0 0 0"/>
-    <geometry name="pioneer_geom">
-      <mesh filename="package://amr_robots_description/meshes/p3at_meshes/${side}_hubcap.stl"/>
+    <child link="p3at_back_${suffix}_axle"/>
+  </joint>
+  <link name="p3at_back_${suffix}_hub">
+    <inertial>
+      <mass value="0.1"/>
+      <origin xyz="0 0 0"/>
+      <inertia ixx="1.0" ixy="0.0" ixz="0.0"
+         iyy="1.0" iyz="0.0" izz="1.0"/>
+      </inertial>
+  <visual name="base_visual">
+    <origin xyz="0 0 0" rpy="0 0 0"/>
+    <geometry name="pioneer_geom">
+      <mesh filename="package://mybot/meshes/p3at_meshes/${suffix}_hubcap.stl"/>
     </geometry>
     <material name="HubcapYellow"/>
@@ -261,28 +294,27 @@
     <origin xyz="0 0 0" rpy="0 0 0"/>
     <geometry>
-      <mesh filename="package://amr_robots_description/meshes/p3at_meshes/${side}_hubcap.stl"/>
-    </geometry>
-  </collision>
-  </link>
-  <gazebo reference="p3at_back_${side}_hub">
+      <mesh filename="package://mybot/meshes/p3at_meshes/${suffix}_hubcap.stl"/>
+    </geometry>
+  </collision>
+  </link>
+  <gazebo reference="p3at_back_${suffix}_hub">
     <material value="Gazebo/Yellow"/>
   </gazebo>
-  <joint name="p3at_back_${side}_hub_joint" type="fixed">
+  <joint name="p3at_back_${suffix}_hub_joint" type="fixed">
     <origin xyz="-0 ${reflect*0.041} 0" rpy="0 0 0"/>
-    <parent link="p3at_back_${side}_axle"/>
-    <child link="p3at_back_${side}_hub"/>
-  </joint>
-  <link name="p3at_back_${side}_wheel">
-    <inertial>
-      <mass value="1.2"/>
+    <parent link="p3at_back_${suffix}_axle"/>
+    <child link="p3at_back_${suffix}_hub"/>
+  </joint>
+  <link name="p3at_back_${suffix}_wheel">
+    <inertial>
+      <mass value="0.5"/>
       <origin xyz="0 0 0"/>
       <inertia ixx="0.012411765597" ixy="0" ixz="0"
-                                                      iyy="0.015218160428" iyz="0"
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